Commit message: Update sancho_ranger.urdf

File: src/sancho_description/urdf/sancho_ranger.urdf (robot description, URDF)
Before this commit: robot ranger_mini_v3, 7 links, 6 joints
Joints:
- joint base_to_laser_back: origin xyz=-0.39 0 0.02 rpy=0 0 3.1415 -> xyz=-0.31 -0.19 0.04 rpy=0 0 2.28761
- joint base_to_laser_front: origin xyz=0.28 0 0.02 rpy=0 0 0 -> xyz=0.31 0.19 0.04 rpy=0 0 -0.785398

Commit message: Update sancho_ranger.urdf

File: src/sancho_description/urdf/sancho_ranger.urdf (robot description, URDF)
Before this commit: robot ranger_mini_v3, 7 links, 6 joints
Joints:
- joint base_to_laser_back: origin xyz=-0.31 -0.19 0.04 rpy=0 0 2.28761 -> xyz=-0.31 0.19 0.04 rpy=0 0 2.28761
- joint base_to_laser_front: origin xyz=0.31 0.19 0.04 rpy=0 0 -0.785398 -> xyz=0.31 -0.19 0.04 rpy=0 0 -0.785398

Commit message: added camera tf and urdf

File: src/sancho_description/urdf/sancho_ranger.urdf (robot description, URDF)
Before this commit: robot ranger_mini_v3, 7 links, 6 joints
Links:
- added link camera_link; visual box size=0.05 0.05 0.05
Joints:
- added joint base_to_camera: type fixed, parent base_link, child camera_link, origin xyz=0.375 0 0.68 rpy=0 0 0

Commit message: Update sancho_ranger.urdf

File: src/sancho_description/urdf/sancho_ranger.urdf (robot description, URDF)
Before this commit: robot ranger_mini_v3, 8 links, 7 joints
Joints:
- joint base_to_laser_back: origin xyz=-0.31 0.19 0.04 rpy=0 0 2.28761 -> xyz=-0.31 0.19 0.04 rpy=0 0 2.35619

Commit message: updated urdf file

File: src/sancho_description/urdf/sancho_ranger.urdf (robot description, URDF)
Before this commit: robot ranger_mini_v3, 8 links, 7 joints
Links:
- added link base_footprint
Joints:
- added joint base_footprint_joint: type fixed, parent base_footprint, child base_link, origin xyz=0 0 0.1 rpy=0 0 0

Commit message: update stl

File: src/sancho_description/urdf/sancho_ranger.urdf (robot description, URDF)
Before this commit: robot ranger_mini_v3, 9 links, 8 joints
Links:
- link base_link: geometry collision mesh filename=package://sancho_description/meshes/ranger_mini3.stl; visual mesh filename=package://sancho_description/meshes/ranger_mini3.stl
- link bl_Link: geometry collision mesh filename=package://sancho_description/meshes/ranger_mini_v3_wheel.stl; visual mesh filename=package://sancho_description/meshes/ranger_mini_v3_wheel.stl
- link fl_Link: geometry collision mesh filename=package://sancho_description/meshes/ranger_mini_v3_wheel.stl; visual mesh filename=package://sancho_description/meshes/ranger_mini_v3_wheel.stl

Commit message: Update sancho_ranger.urdf

File: src/sancho_description/urdf/sancho_ranger.urdf (robot description, URDF)
Before this commit: robot ranger_mini_v3, 9 links, 8 joints
Joints:
- joint base_footprint_joint: origin xyz=0 0 0.1 rpy=0 0 0 -> xyz=0 0 0.325 rpy=0 0 0

Commit message: Update sancho_ranger.urdf

File: src/sancho_description/urdf/sancho_ranger.urdf (robot description, URDF)
Before this commit: robot ranger_mini_v3, 9 links, 8 joints
Links:
- link bl_Link: geometry collision mesh filename=package://sancho_description/meshes/ranger_mini_v3_wheel.dae; visual mesh filename=package://sancho_description/meshes/ranger_mini_v3_wheel.dae
- link fl_Link: geometry collision mesh filename=package://sancho_description/meshes/ranger_mini_v3_wheel.dae; visual mesh filename=package://sancho_description/meshes/ranger_mini_v3_wheel.dae

Commit message: Update sancho_ranger.urdf

File: src/sancho_description/urdf/sancho_ranger.urdf (robot description, URDF)
Before this commit: robot ranger_mini_v3, 9 links, 8 joints
Links:
- added link body_link; collision box size=0.01 0.2 0.68; visual box size=0.01 0.2 0.68
- added link head_link; collision box size=0.205 0.125 0.1; visual box size=0.205 0.125 0.1
- added link neck_link; collision cylinder length=0.05 radius=0.0525; visual cylinder length=0.05 radius=0.0525
Joints:
- added joint body_link_joint: type fixed, parent base_link, child body_link, origin xyz=0 0 0 rpy=0 0 0
- added joint body_to_neck: type fixed, parent body_link, child neck_link, origin xyz=0 0 0 rpy=0 0 0
- added joint neck_to_head: type fixed, parent neck_link, child head_link, origin xyz=0 0 0 rpy=0 0 0

Commit message: Update sancho_ranger.urdf

File: src/sancho_description/urdf/sancho_ranger.urdf (robot description, URDF)
Before this commit: robot ranger_mini_v3, 12 links, 11 joints
Links:
- link body_link: geometry collision box size=0.4 0.32 0.7; visual box size=0.4 0.32 0.7

Commit message: Fix ptu tf and joins

File: src/sancho_description/urdf/sancho_ranger.urdf (robot description, URDF)
Before this commit: robot ranger_mini_v3, 12 links, 11 joints
Links:
- removed link neck_link
- added link turret_pan_link; visual cylinder length=0.08 radius=0.04
- added link turret_tilt_link; visual box size=0.05 0.1 0.025
- link head_link: geometry visual box size=0.205 0.125 0.1
Joints:
- removed joint body_to_neck
- removed joint neck_to_head
- added joint pan: type revolute, parent body_link, child turret_pan_link, origin xyz=0.22 0 0.725 rpy=0 0 0, axis 0 0 1, limit lower=-3.14 upper=3.14 effort=1.0 velocity=1.0
- added joint tilt: type revolute, parent turret_pan_link, child turret_tilt_link, origin xyz=0 0 0.05 rpy=0 0 0, axis 0 1 0, limit lower=-1.57 upper=1.57 effort=1.0 velocity=1.0
- added joint tilt_to_head: type fixed, parent turret_tilt_link, child head_link, origin xyz=0 0 0 rpy=0 0 0
